File: kicad/automato-eink/automato-eink.kicad_pcb (KiCad board)
At the start: 2 copper layers, 62.5 x 35 mm, 23 parts, among them J1 Conn_01x24, J2 Conn_01x08_Male, Q1 Q_NMOS_GDS

Commit message: add standoffs
Parts:
- added REF**: MountingHole_2.2mm_M2_DIN965_Pad_TopBottom, MountingHole:MountingHole_2.2mm_M2_DIN965_Pad_TopBottom, F.Cu at (139.8, 122.8)
- added REF**: MountingHole_2.2mm_M2_DIN965_Pad_TopBottom, MountingHole:MountingHole_2.2mm_M2_DIN965_Pad_TopBottom, F.Cu at (139.8, 92.2)
